File: PIC32-SSOP28-Breakout/PCI32-SSOP28.kicad_pcb (KiCad board)
At the start: 2 copper layers, 33 x 15.2 mm, 17 parts, among them CN1 CONN_12, CN2 CONN_12, J1 JMP, U1 PIC32MMXXXXGPL028, X1 NX3225-8M, X2 32.768k

Commit message: fix silk typo
Other:
- board text added: "RB3"
Changed lines of the file:
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@@
 (kicad_pcb (version 4) (host pcbnew 4.0.6)
   (general
-    (links 61)
-    (no_connects 6)
-    (area 133.274999 97.714999 166.445001 113.105001)
+    (links 56)
+    (no_connects 0)
+    (area 133 92.23 177.220922 114.675)
     (thickness 1.6)
     (drawings 38)
@@
   (title_block
     (title PIC32MM_breakout)
-    (date 2017-04-22)
-    (rev B)
+    (date 2017-09-20)
+    (rev c)
     (company "Kent_Nakazawa ( kent_n@outlook.com )")
   )
@@
     (effects (font (size 0.8 0.8) (thickness 0.15)) (justify left mirror))
   )
-  (gr_text RA3 (at 152.45 107.93 90) (layer B.SilkS)
-    (effects (font (size 0.8 0.8) (thickness 0.15)) (justify left mirror))
-  )
-  (gr_text RA2 (at 149.85 107.93 90) (layer B.SilkS)
-    (effects (font (size 0.8 0.8) (thickness 0.15)) (justify left mirror))
-  )
+  (gr_text RA2 (at 152.45 107.93 90) (layer B.SilkS)
+    (effects (font (size 0.8 0.8) (thickness 0.15)) (justify left mirror))
+  )
+  (gr_text RB3 (at 149.85 107.93 90) (layer B.SilkS)
+    (effects (font (size 0.8 0.8) (thickness 0.15)) (justify left mirror))
+  )
